Commit message: Update landmark dimensions acording to the specification

File: leo_erc_gazebo_worlds/sdf/landmark.sdf.xacro (robot description, xacro)
@@ -2,8 +2,8 @@
 <sdf version="1.6" xmlns:xacro="http://www.ros.org/wiki/xacro">
   <xacro:macro name="landmark" params="id *pose">
-    <xacro:property name="pole_above_ground" value="0.1"/>
+    <xacro:property name="pole_above_ground" value="0.3"/>
+    <xacro:property name="box_width" value="0.25"/>
     <xacro:property name="pole_below_ground" value="0.1"/>
-    <xacro:property name="box_width" value="0.24"/>
-    <xacro:property name="box_height" value="0.34"/>
+    <xacro:property name="box_height" value="0.32"/>
     <xacro:property name="sheet_width" value="0.005"/> <!-- When the sheet is too thin it is not shaded properly for some reason -->
     <xacro:property name="sheet_out" value="0.001"/>
@@ -15,7 +15,8 @@
           <pose>0 0 ${(pole_above_ground - pole_below_ground)/2} 0 0 0</pose>
           <geometry>
-            <box>
-              <size>0.05 0.02 ${pole_above_ground + pole_below_ground}</size>
-            </box>
+            <cylinder>
+              <radius>0.01</radius>
+              <length>${pole_above_ground + pole_below_ground}</length>
+            </cylinder>
           </geometry>
           <material>
@@ -28,7 +29,8 @@
           <pose>0 0 ${(pole_above_ground - pole_below_ground)/2} 0 0 0</pose>
           <geometry>
-            <box>
-              <size>0.05 0.02 ${pole_above_ground + pole_below_ground}</size>
-            </box>
+            <cylinder>
+              <radius>0.01</radius>
+              <length>${pole_above_ground + pole_below_ground}</length>
+            </cylinder>
           </geometry>
         </collision>
